File: circuit/FM1216.kicad_sch (KiCad schematic)
At the start: 61 parts, among them J1 DE9_Pins, J2 AudioJack, Q1 BC850, SW1 RotaryEncode, SW2 REREAD, U1 PIC16F876-XXISO, U2 MAX232, U3 PCF8574T, U4 L7805, Y1 20MHz

Commit message: next generation v1
Parts:
- removed R9: 10k, symbol Device:R
- removed SW2: REREAD, symbol Switch:SW_DPST_x2
- added J3: Conn_01x08_Pin, symbol Connector:Conn_01x08_Pin
- added J4: Conn_01x08_Socket, symbol Connector:Conn_01x08_Socket
- added SW10: '7', symbol Switch:SW_Push
- added SW11: '8', symbol Switch:SW_Push
- added SW12: '9', symbol Switch:SW_Push
- added SW13: 'C', symbol Switch:SW_Push
- added SW14: '*', symbol Switch:SW_Push
- added SW15: '0', symbol Switch:SW_Push
- added SW16: '#', symbol Switch:SW_Push
- added SW17: 'D', symbol Switch:SW_Push
- added SW2: '1', symbol Switch:SW_Push
- added SW3: '2', symbol Switch:SW_Push
- added SW4: `3`, symbol Switch:SW_Push
- added SW5: 'A', symbol Switch:SW_Push
- added SW6: '4', symbol Switch:SW_Push
- added SW7: '5', symbol Switch:SW_Push
- added SW8: '6', symbol Switch:SW_Push
- added SW9: 'B', symbol Switch:SW_Push
Connections:
- net C1: now reaches U1.21 (INT/RB0)
- net C1: now also J3.1 (Pin_1), J4.1 (Pin_1), SW10.2, SW14.2, SW2.2, SW6.2
- net C2: now reaches U1.22 (RB1)
- net C2: now also J3.2 (Pin_2), J4.2 (Pin_2), SW11.2, SW15.2, SW3.2, SW7.2
- net C3: now reaches U1.23 (RB2)
- net C3: now also J3.3 (Pin_3), J4.3 (Pin_3), SW12.2, SW16.2, SW4.2, SW8.2
- net C4: now reaches U1.24 (PGM/RB3)
- net C4: now also J3.4 (Pin_4), J4.4 (Pin_4), SW13.2, SW17.2, SW5.2, SW9.2
- net R1: now reaches U1.25 (RB4)
- net R1: now also J3.5 (Pin_5), J4.5 (Pin_5), SW2.1, SW3.1, SW4.1, SW5.1
- net R2: now reaches U1.26 (RB5)
- net R2: now also J3.6 (Pin_6), J4.6 (Pin_6), SW6.1, SW7.1, SW8.1, SW9.1
- net R3: now reaches U1.27 (PGC/RB6)
- net R3: now also J3.7 (Pin_7), J4.7 (Pin_7), SW10.1, SW11.1, SW12.1, SW13.1
- net R4: now reaches U1.28 (PGD/RB7)
- net R4: now also J3.8 (Pin_8), J4.8 (Pin_8), SW14.1, SW15.1, SW16.1, SW17.1
Other:
- moved on the sheet: AE1, C1, C10, C11, C12, C13, C14, C15, C16, C17, C18, C19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

Commit message: Fix circuit
Changed lines of the file:
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@@
 	(wire
 		(pts
+			(xy 251.46 59.69) (xy 251.46 60.96)
+		)
+		(stroke
+			(width 0)
+			(type default)
+		)
+	)
+	(wire
+		(pts
 			(xy 220.98 142.24) (xy 226.06 142.24)
 		)
@@
 					(unit 1)
 				)
+			)
+		)
+	)
+	(symbol
+		(lib_id "power:GNDD")
+		(at 251.46 60.96 0)
+		(mirror y)
+		(unit 1)
+		(exclude_from_sim no)
+		(in_bom yes)
+		(on_board yes)
+		(dnp no)
+		(fields_autoplaced yes)
+		(property "Reference" "#PWR03"
+			(at 251.46 67.31 0)
+			(effects
+				(font
+					(size 1.27 1.27)
+				)
+				(hide yes)
+			)
+		)
+		(property "Value" "GND"
+			(at 251.46 64.77 0)
+			(effects
+				(font
+					(size 1.27 1.27)
+				)
+			)
+		)
+		(property "Footprint" ""
+			(at 251.46 60.96 0)
+			(effects
+				(font
+					(size 1.27 1.27)
+				)
+				(hide yes)
+			)
+		)
+		(property "Datasheet" ""
+			(at 251.46 60.96 0)
+			(effects
+				(font
+					(size 1.27 1.27)
+				)
+				(hide yes)
+			)
+		)
+		(property "Description" "Power symbol creates a global label with name \"GNDD\" , digital ground"
+			(at 251.46 60.96 0)
+			(effects
+				(font
+					(size 1.27 1.27)
+				)
+				(hide yes)
+			)
+		)
+		(pin "1"
+		)
+		(instances
+			(project "FM1216"
+				(path "/65cde581-a21d-47f8-a0b3-e48af637757e"
+					(reference "#PWR03")
+					(unit 1)
+				)
